File: hw/remote-pallet/remote-pallet.sch (KiCad schematic (older format))
At the start: 26 parts, among them J1 Power, M0 E-MATCH, M1 E-MATCH, M2 E-MATCH, M3 E-MATCH, M4 E-MATCH, M5 E-MATCH, M6 E-MATCH, M7 E-MATCH, Q1 EMatch Test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

Commit message: updaint schematic and layout
Connections:
- net Armed: now also U2.20 (D7); no longer U2.4 (RX)
- net SenseSwitch: now also U2.4 (RX); no longer U2.20 (D7)
Changed lines of the file:
@@
 Text GLabel 1550 3300 0    60   Input ~ 0
 Sense7
+Text GLabel 3150 3000 2    60   Input ~ 0
+SenseSwitch
 Text GLabel 3150 3500 2    60   Input ~ 0
-SenseSwitch
-Text GLabel 3150 3000 2    60   Input ~ 0
 Armed
 Text GLabel 1550 3100 0    60   Input ~ 0
